File: BM_Solar_V1-1.kicad_pcb (KiCad board)
At the start: 2 copper layers, 21.1 x 40.9 mm, 20 parts, among them J1 LiPo, J10 Conn_01x16_Pin, J2 LiFePO4, J4 1S Batt 1A, J5 Thrm - 10k, J8 Conn_01x16_Pin, J9 Solar 3-18V, U1 BQ25185DLHR

Commit message: Changed to a 1x3 pin header for battery select, rearranged batt sense circuit, improved traces, and added more vias for more thermal dissipation.
Parts:
- removed J1: LiPo, Connector_PinHeader_2.54mm:PinHeader_1x02_P2.54mm_Vertical
- removed J2: LiFePO4, Connector_PinHeader_2.54mm:PinHeader_1x02_P2.54mm_Vertical
- added J3: Batt Sel, Connector_PinHeader_2.54mm:PinHeader_1x03_P2.54mm_Vertical, F.Cu at (139.9, 112.7)
- J4: value 1S Batt 1A -> Batt 1S
- U1: footprint footprints:WSON10_DLH_TEX -> bq25185 footprints:WSON10_DLH_TEX
- moved G*** 9.95 mm to (132.6, 112.3)
- moved R3 7.34 mm to (131.3, 100.0)
- moved R4 7.34 mm to (131.3, 102.3)
Routing:
- net Net-(J4-Pin_1): track 26.1 -> 18.8 mm
- net Net-(J3-Pin_2): track 18.1 -> 15.2 mm
- net Net-(J5-Pin_1): track 24.1 -> 22.4 mm
- net Net-(J8-Pin_10): track 8.10 -> 6.98 mm
- net Net-(J3-Pin_3): track 4.45 -> 3.84 mm
- net GND: track 28.1 -> 28.4 mm, vias 40 -> 116
Other:
- board text added: "LiFePO4"
- board text added: "LiIon/ LiPo"
- board text added: "__"
